File: LightMinderSMD.kicad_sch (KiCad schematic)
At the start: 32 parts, among them J1 Conn_01x04_Female, J3 Conn_01x04, J4 Conn_01x02_Female, Q1 Q_NPN_BEC, Q2 Q_NPN_BEC, Q3 STD35P6LLF6, U2 LM3480-3.3

Commit message: ICSP Typo Fix
Parts:
- D7: footprint SamacSys_Parts:DO-214ACSMA -> Diode_SMD:D_SMA
Changed lines of the file:
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@@
       (effects (font (size 1.27 1.27)) (justify left))
     )
-    (property "Footprint" "SamacSys_Parts:DO-214ACSMA" (id 2) (at 233.68 77.47 0)
+    (property "Footprint" "Diode_SMD:D_SMA" (id 2) (at 233.68 77.47 0)
       (effects (font (size 1.27 1.27)) hide)
     )
@@
     (pin "3")
   )
-  (symbol (lib_id "Device:R") (at 232.41 26.67 0)
+  (symbol (lib_id "Device:R") (at 232.41 26.67 0) (unit 1)
     (in_bom yes) (on_board yes)
     (property "Reference" "R13" (id 0) (at 234.188 25.5016 0)
@@
     (pin "2")
   )
-  (symbol (lib_id "Device:LED") (at 232.41 36.83 90)
+  (symbol (lib_id "Device:LED") (at 232.41 36.83 90) (unit 1)
     (in_bom yes) (on_board yes)
     (property "Reference" "D8" (id 0) (at 235.3818 35.8394 90)
@@
     (pin "2")
   )
-  (symbol (lib_id "Device:R") (at 219.71 26.67 0)
+  (symbol (lib_id "Device:R") (at 219.71 26.67 0) (unit 1)
     (in_bom yes) (on_board yes)
     (property "Reference" "R11" (id 0) (at 221.488 25.5016 0)
@@
     (pin "2")
   )
-  (symbol (lib_id "Device:LED") (at 219.71 36.83 90)
+  (symbol (lib_id "Device:LED") (at 219.71 36.83 90) (unit 1)
     (in_bom yes) (on_board yes)
     (property "Reference" "D6" (id 0) (at 222.6818 35.8394 90)
@@
     (pin "2")
   )
-  (symbol (lib_id "Device:R") (at 245.11 26.67 0)
+  (symbol (lib_id "Device:R") (at 245.11 26.67 0) (unit 1)
     (in_bom yes) (on_board yes)
     (property "Reference" "R14" (id 0) (at 246.888 25.5016 0)
@@
     (pin "2")
   )
-  (symbol (lib_id "Device:LED") (at 245.11 36.83 90)
+  (symbol (lib_id "Device:LED") (at 245.11 36.83 90) (unit 1)
     (in_bom yes) (on_board yes)
     (property "Reference" "D9" (id 0) (at 248.0818 35.8394 90)
@@
     (pin "2")
   )
-  (symbol (lib_id "Device:R") (at 257.81 26.67 0)
+  (symbol (lib_id "Device:R") (at 257.81 26.67 0) (unit 1)
     (in_bom yes) (on_board yes)
     (property "Reference" "R15" (id 0) (at 259.588 25.5016 0)
@@
     (pin "2")
   )
-  (symbol (lib_id "Device:LED") (at 257.81 36.83 90)
+  (symbol (lib_id "Device:LED") (at 257.81 36.83 90) (unit 1)
     (in_bom yes) (on_board yes)
     (property "Reference" "D10" (id 0) (at 260.7818 35.8394 90)
@@
     (pin "2")
   )
-  (symbol (lib_id "power:GND") (at 238.76 44.45 0)
+  (symbol (lib_id "power:GND") (at 238.76 44.45 0) (unit 1)
     (in_bom yes) (on_board yes)
     (property "Reference" "#PWR0105" (id 0) (at 238.76 50.8 0)
@@
     (pin "2")
   )
-  (symbol (lib_id "Device:C") (at 59.69 88.9 0)
+  (symbol (lib_id "Device:C") (at 59.69 88.9 0) (unit 1)
     (in_bom yes) (on_board yes)
     (property "Reference" "C5" (id 0) (at 62.611 87.7316 0)
@@
     (pin "2")
   )
-  (symbol (lib_id "Device:C") (at 58.42 124.46 0)
+  (symbol (lib_id "Device:C") (at 58.42 124.46 0) (unit 1)
     (in_bom yes) (on_board yes)
     (property "Reference" "C9" (id 0) (at 61.341 123.2916 0)
@@
     )
     (path "/00000000-0000-0000-0000-0000618e275a"
-      (reference "D7") (unit 1) (value "20v TVS") (footprint "SamacSys_Parts:DO-214ACSMA")
+      (reference "D7") (unit 1) (value "20v TVS") (footprint "Diode_SMD:D_SMA")
     )
     (path "/00000000-0000-0000-0000-0000618fd117"
